Commit message: start creating the joints

File: public/ufactory_description/lite6/urdf/lite6.urdf (robot description, URDF)
Before this commit: robot lite6, 9 links, 8 joints
Links:
- link link1: geometry collision mesh filename=../meshes/collision/link1.stl; visual mesh filename=../meshes/visual/link1.stl
- link link2: geometry collision mesh filename=../meshes/collision/link2.stl; visual mesh filename=../meshes/visual/link2.stl
- link link3: geometry collision mesh filename=../meshes/collision/link3.stl; visual mesh filename=../meshes/visual/link3.stl
- link link4: geometry collision mesh filename=../meshes/collision/link4.stl; visual mesh filename=../meshes/visual/link4.stl
- link link5: geometry collision mesh filename=../meshes/collision/link5.stl; visual mesh filename=../meshes/visual/link5.stl
- link link6: geometry collision mesh filename=../meshes/collision/link6.stl; visual mesh filename=../meshes/visual/link6.stl
- link link_base: geometry collision mesh filename=../meshes/collision/base.stl; visual mesh filename=../meshes/visual/base.stl
- link link_eef: geometry collision mesh filename=../meshes/collision/gripper_lite.stl; visual mesh filename=../meshes/visual/gripper_lite.stl
